Commit message: Update wall.urdf

File: simple_driving/resources/wall.urdf (robot description, URDF)
Before this commit: robot wall, 1 links, 0 joints
Links:
- link base_link: geometry collision box size=1 10 1; visual box size=1 10 1

Commit message: Update wall.urdf

File: simple_driving/resources/wall.urdf (robot description, URDF)
Before this commit: robot wall, 1 links, 0 joints
Links:
- link base_link: geometry collision cylinder length=1 radius=0.5; visual cylinder length=1 radius=0.5
